File: Project NuXT.sch (KiCad schematic (older format))
At the start: 198 parts, among them P1 CF Connector, P10 IDE, P2 Triple_D-sub_PC99, P3 Speaker, P4 VGA Rear Port, P5 Floppy, P6 PC/104 Platform, P7 ATX Power, P8 Front Panel, P9 StackedMini-DIN-6, Q1 MMBT3904, Q2 MMBT3904, SW1 System Config, SW2 UMB Config, SW3 COM Port Config, SW4 Mouse Port Config, SW5 Parallel Port Config, SW6 Power, SW7 Reset, U1 8088, U10 PIC12F629, U11 ATtiny2313, U12 HC138, U13 AHC32, U14 HC04, U15 AHCT573, U16 AHCT245, U17 HC138, U18 HC08, U19 AHCT573, U2 8087, U20 AHCT245, U21 75232, U22 HC04, U23 HC138, U24 HC08, U25 AHCT573, U26 AHCT245, U27 555, U28 AHC32, U29 AHCT245, U3 FE2010A, U30 7905, U31 AC11, U32 HC138, U33 HC138, U34 HC04, U35 AHCT573, U36 AHCT245, U37 AHCT573, U4 AS6C4008, U5 AS6C4008, U6 SST39SF010A, U7 TL16C552AFN, U8 PC8477, U9 DS12885, X1 1.8432MHz, Y1 32.768kHz 6pF, Y2 24MHz, Y3 28.63636MHz, Y4 8MHz

Commit message: Add files via upload
Parts:
- C1, C2: LCSC P# C1710 -> (none)
- C10, C11, C3, C4, C6: LCSC P# C1804 -> (none)
- C12, C13, C14, C15, C16, C17, C18, C19, C20, C21, C22, C23, C24, C25, C26, C27, C28, C29, C30, C31, C32, C33, C34, C35, C36, C37, C38, C39, C40, C41, C52, C55, C60, C61, C62, C63, C65, C66, C67, C68, C69, C70, C71: LCSC P# C14663 -> (none)
- C42, C43, C44, C45, C46, C47, C48, C49, C50, C51, C58, C64, C7: LCSC P# C19702 -> (none)
- C5: LCSC P# C14857 -> (none)
- C53, C54, C56, C57: LCSC P# C15850 -> (none)
- C8: LCSC P# C28323 -> (none)
- D1: LCSC P# C417352 -> (none)
- D2: LCSC P# C84256 -> (none)
- D3: LCSC P# C72038 -> (none)
- D4: LCSC P# C72043 -> (none)
- D5: LCSC P# C409769 -> (none)
- D6: LCSC P# C81598 -> (none)
- F1, F2: LCSC P# C163516 -> (none)
- Q1, Q2: LCSC P# C20526 -> (none)
- R1, R2, R20, R4, R5, R6: LCSC P# C17634 -> (none)
- R10: LCSC P# C17514 -> (none)
- R11, R12, R13, R14, R15, R16, R17, R18, R19, R3, R7, R9: LCSC P# C17513 -> (none)
- R21, R22, R8: LCSC P# C17407 -> (none)
- RN1, RN13, RN4, RN5: LCSC P# C1980 -> (none)
- RN10, RN11, RN12, RN2, RN3, RN6, RN7, RN8: LCSC P# C29718 -> (none)
- SW6, SW7: LCSC P# C128536 -> (none)
- U11: LCSC P# C22281 -> (none)
- U12, U17, U23, U32, U33: LCSC P# C5602 -> (none)
- U13, U28: LCSC P# C7490 -> (none)
- U14, U22, U34: LCSC P# C5590 -> (none)
- U15, U19, U25, U35, U37: LCSC P# C282327 -> (none)
- U16, U20, U26, U29, U36: LCSC P# C173388 -> (none)
- U18, U24: LCSC P# C5593 -> (none)
- U21: LCSC P# C171524 -> (none)
- U27: LCSC P# C7593 -> (none)
- U30: LCSC P# C75505 -> (none)
- U31: LCSC P# C327489 -> (none)
- Y1: LCSC P# C94673 -> (none)
- Y2: symbol 8088-FE2010A-SBC-rescue:Crystal_Small -> Device:Crystal_Small; LCSC P# C112570 -> (none)
- Y3: symbol 8088-FE2010A-SBC-rescue:Crystal_Small -> Device:Crystal_Small; LCSC P# C112564 -> (none)
- Y4: LCSC P# C115962 -> (none)
